Commit message: gazebo start

File: description/robot_core.xacro (robot description, xacro)
@@ -50,4 +50,7 @@
         </xacro:inertial_box>
     </link>
+    <gazebo reference="chassis">
+        <material>Gazebo/White</material>
+    </gazebo>
 <!--===============================================================================================-->
     <!-- LEFT WHEEL -->
@@ -75,4 +78,7 @@
         </xacro:inertial_cylinder>
     </link>
+    <gazebo reference="left_wheel">
+        <material>Gazebo/Blue</material>
+    </gazebo>
 <!--===============================================================================================-->
     <!-- RIGHT WHEEL -->
@@ -100,4 +106,7 @@
         </xacro:inertial_cylinder>
     </link>
+    <gazebo reference="right_wheel">
+        <material>Gazebo/Blue</material>
+    </gazebo>
 <!--===============================================================================================-->
     <!-- CASTER WHEEL -->
@@ -124,3 +133,6 @@
         </xacro:inertial_sphere>
     </link>
+    <gazebo reference="caster_wheel">
+        <material>Gazebo/Black</material>
+    </gazebo>
 </robot>
